File: pcb/bw_beer_caddy/bw_beer_caddy.kicad_sch (KiCad schematic)
At the start: 34 parts, among them J1 Screw_Terminal_01x06, J3 Screw_Terminal_01x03, J4 Screw_Terminal_01x03, J5 Conn_01x03_Female, J6 Conn_01x03_Female, J7 Conn_02x04_Top_Bottom, J8 Conn_02x04_Top_Bottom, J9 Screw_Terminal_01x06, K1 G5LE-1, Q1 2N3904, Q2 FQP27P06, Q3 2N7000, Q4 2N3904, Q5 2N7000, U1 ina219_breakout, U2 LM2575-5.0BT, U3 LM2575-12BT, U4 LM2575-12BT, U5 LM2575-12BT, U6 SEN-13879

Commit message: bw_bcause rev 00 release
Parts:
- removed J3, J4: Screw_Terminal_01x03, TerminalBlock_TE-Connectivity:TerminalBlock_TE_282834-3_1x03_P2.54mm_Horizontal, symbol Connector:Screw_Terminal_01x03
- removed J7: Conn_02x04_Top_Bottom, Connector_PinHeader_2.54mm:PinHeader_2x04_P2.54mm_Vertical, symbol Connector_Generic:Conn_02x04_Top_Bottom
- removed R2: 30K, Resistor_SMD:R_0805_2012Metric, symbol Device:R_US
- removed R4: 10K, Resistor_SMD:R_0805_2012Metric, symbol Device:R_US
- removed U3, U4, U5: LM2575-12BT, Package_TO_SOT_THT:TO-220-5_Vertical, symbol Regulator_Switching:LM2575-12BT
- added D2, D3, D4: LED, LED_SMD:LED_1206_3216Metric, symbol Device:LED
- added J10, J2: Conn_01x03_Female, Connector_PinHeader_2.54mm:PinHeader_1x03_P2.54mm_Vertical, symbol Connector:Conn_01x03_Female
- added J3: Screw_Terminal_01x04, TerminalBlock_TE-Connectivity:TerminalBlock_TE_282834-4_1x04_P2.54mm_Horizontal, symbol Connector:Screw_Terminal_01x04
- added J4: Screw_Terminal_01x05, TerminalBlock_TE-Connectivity:TerminalBlock_TE_282834-5_1x05_P2.54mm_Horizontal, symbol Connector:Screw_Terminal_01x05
- added J7: Conn_02x08_Top_Bottom, Connector_PinHeader_2.54mm:PinHeader_2x08_P2.54mm_Vertical, symbol Connector_Generic:Conn_02x08_Top_Bottom
- added R10, R11, R12, R13: 10K, Resistor_SMD:R_0805_2012Metric, symbol Device:R_US
- added U3, U4, U5: LM2576TV-012G, Package_TO_SOT_THT:TO-220-5_P3.4x3.7mm_StaggerOdd_Lead3.8mm_Vertical, symbol bwbots:LM2576TV-012G
- R8: value 6K -> 10K
Connections:
- net +12L: now also U3.2 (OUTPUT)
- net +12V: now also U4.2 (OUTPUT), U5.2 (OUTPUT)
- net +3.3V: now also U1.1 (VCC), J10.3 (Pin_3), J7.1 (Pin_1), J7.13 (Pin_13), J7.5 (Pin_5), J7.9 (Pin_9), R10.2, R13.2; no longer U1. (VIN-)
- net +5V: now also J4.1 (Pin_1), J4.3 (Pin_3)
- net CHARGE_RELAY_CTRL: now also U$2.29
- net GND: now also U1.2 (GND), D2.1 (K), D3.1 (K), D4.1 (K), J10.2 (Pin_2), J2.3 (Pin_3), J3.2 (Pin_2), J3.4 (Pin_4), J4.2 (Pin_2), J4.4 (Pin_4), J7.12 (Pin_12), J7.16 (Pin_16), J7.4 (Pin_4), J7.8 (Pin_8), U3.3 (GND), U4.3 (GND), U5.3 (GND); no longer U1. (VIN-)
- net LATCH_OUT: now also U1.6 (VIN+); no longer U1. (VIN-)
- net LATCH_STAT: now also U$2.31/A12; no longer U$2.25
- net LED_RING: now also J4.5 (Pin_5)
- net M1_EA: now also U$2.3/CANTX, J7.2 (Pin_2); no longer U$2.23/A9
- net M1_EB: now also U$2.4/CANRX, J7.3 (Pin_3); no longer U$2.22/A8
- net M2_EA: now also U$2.5, J7.6 (Pin_6), J7.7 (Pin_7); no longer U$2.21/A7
- net M2_EB: now also U$2.6; no longer U$2.20/A6
- net M3_DR1: now also U$2.23/A9; no longer U$2.27
- net M3_DR2: now also U$2.22/A8; no longer U$2.28
- net M3_EA: now also U$2.24, J7.10 (Pin_10); no longer U$2.3/CANTX
- net M3_EB: now also U$2.25, J7.11 (Pin_11); no longer U$2.4/CANRX
- net M4_DR1: now also U$2.21/A7; no longer U$2.29
- net M4_DR2: now also U$2.20/A6; no longer U$2.30
- net M4_EA: now also U$2.26, J7.14 (Pin_14); no longer U$2.5
- net M4_EB: now also U$2.27, J7.15 (Pin_15); no longer U$2.6
- net MOTOR_ENABLE: now also U$2.33/A14, R11.2, U4.5 (*ON/OFF), U5.5 (*ON/OFF); no longer U$2.8
- net RX_JETSON: now also U$2.7, J2.2 (Pin_2); no longer U$2.33/A14
- net SCL1: now also U1.3 (SCL); no longer U1. (VIN-)
- net SDA1: now also U1.4 (SDA); no longer U1. (VIN-)
- net TX_JETSON: now also U$2.8, J2.1 (Pin_1); no longer U$2.34/A15
- net UNLATCH: now also U$2.30; no longer U$2.24
- net USB_SENSE: now also U$2.34/A15; no longer U$2.7
- net VDD: now also U1.5 (VIN-), U3.1 (VIN), U4.1 (VIN), U5.1 (VIN); no longer U1. (VIN-)
- net HALL_EFFECT_SNS: now reaches U$2.17/A3
- net HALL_EFFECT_SNS: now also J10.1 (Pin_1), R13.1
- net STATUS_LED: now reaches U$2.32/A13
- net STATUS_LED: now also R12.2
- net at K1.1: now also J3.1 (Pin_1), J3.3 (Pin_3)
- new net: D3.2 (A), R11.1
- new net: D2.2 (A), R10.1
- new net: D4.2 (A), R12.1

Commit message: pcb rev 01 08-21-2022
Parts:
- removed C1, C2: 22 UF, Capacitor_THT:C_Disc_D5.0mm_W2.5mm_P5.00mm, symbol Device:C
- removed D1: 1N5822, Diode_THT:D_DO-201AD_P15.24mm_Horizontal, symbol Diode:1N5822
- removed J1, J9: Screw_Terminal_01x06, TerminalBlock_TE-Connectivity:TerminalBlock_TE_282834-6_1x06_P2.54mm_Horizontal, symbol Connector:Screw_Terminal_01x06
- removed J2: Conn_01x03_Female, Connector_PinHeader_2.54mm:PinHeader_1x03_P2.54mm_Vertical, symbol Connector:Conn_01x03_Female
- removed J3: Screw_Terminal_01x04, TerminalBlock_TE-Connectivity:TerminalBlock_TE_282834-4_1x04_P2.54mm_Horizontal, symbol Connector:Screw_Terminal_01x04
- removed J4: Screw_Terminal_01x05, TerminalBlock_TE-Connectivity:TerminalBlock_TE_282834-5_1x05_P2.54mm_Horizontal, symbol Connector:Screw_Terminal_01x05
- removed J7: Conn_02x08_Top_Bottom, Connector_PinHeader_2.54mm:PinHeader_2x08_P2.54mm_Vertical, symbol Connector_Generic:Conn_02x08_Top_Bottom
- removed J8: Conn_02x04_Top_Bottom, Connector_PinHeader_2.54mm:PinHeader_2x04_P2.54mm_Vertical, symbol Connector_Generic:Conn_02x04_Top_Bottom
- removed K1: G5LE-1, Relay_THT:Relay_SPDT_Omron-G5LE-1, symbol Relay:G5LE-1
- removed Q1, Q4: 2N3904, Package_TO_SOT_THT:TO-92_Inline, symbol Transistor_BJT:2N3904
- removed Q2: FQP27P06, Package_TO_SOT_THT:TO-220-3_Vertical, symbol Transistor_FET:FQP27P06
- removed Q3, Q5: 2N7000, Package_TO_SOT_THT:TO-92_Inline, symbol Transistor_FET:2N7000
- removed R1, R13, R3, R5, R8, R9: 10K, Resistor_SMD:R_0805_2012Metric, symbol Device:R_US
- removed R6: 100K, Resistor_SMD:R_0805_2012Metric, symbol Device:R_US
- removed R7: 10 Ohm, Resistor_THT:R_Axial_DIN0207_L6.3mm_D2.5mm_P10.16mm_Horizontal, symbol Device:R_US
- removed U$1: PCA9685, bwbots:PCA9685, symbol bwbots:PCA9685
- removed U1: ina219_breakout, bwbots:ina219_breakout, symbol bwbots:ina219_breakout
- removed U2: LM2575-5.0BT, Package_TO_SOT_THT:TO-220-5_Vertical, symbol Regulator_Switching:LM2575-5.0BT
- removed U3, U4, U5: LM2576TV-012G, Package_TO_SOT_THT:TO-220-5_P3.4x3.7mm_StaggerOdd_Lead3.8mm_Vertical, symbol bwbots:LM2576TV-012G
- removed U6: SEN-13879, SPARKFUN_SEN-13879, symbol bwbots:SEN-13879
- added J1, J12, J2, J3, J4, J8, J9: Conn_01x04_Female, Connector_JST:JST_XH_B4B-XH-A_1x04_P2.50mm_Vertical, symbol Connector:Conn_01x04_Female
- added J11, J13, J7: Conn_01x03_Female, Connector_JST:JST_XH_B3B-XH-A_1x03_P2.50mm_Vertical, symbol Connector:Conn_01x03_Female
- added J14: Conn_01x02_Female, Connector_PinHeader_2.54mm:PinHeader_1x02_P2.54mm_Vertical, symbol Connector:Conn_01x02_Female
- added J15: Conn_01x02_Female, TerminalBlock_4Ucon:TerminalBlock_4Ucon_1x02_P3.50mm_Horizontal, symbol Connector:Conn_01x02_Female
- added U1: Pololu_5V_Step_Down_2851, bwbots:Pololu_5V_Step_Down_2851, symbol bwbots:Pololu_5V_Step_Down_2851
- added U2, U3: Pololu-MC33926-Dual-Motor, bwbots:Pololu-MC33926-Dual-Motor-Vertical, symbol bwbots:Pololu-MC33926-Dual-Motor
- D1: renamed from D2; Part Number (none) -> 1078
- D2: renamed from D3; Part Number (none) -> 1078
- D3: renamed from D4; Part Number (none) -> 1078
- J10, J5, J6: footprint Connector_PinHeader_2.54mm:PinHeader_1x03_P2.54mm_Vertical -> Connector_JST:JST_XH_B3B-XH-A_1x03_P2.50mm_Vertical; Part Number (none) -> 1083
- R1: renamed from R10; Part Number (none) -> 1090
- R2: renamed from R11; Part Number (none) -> 1090
- R3: renamed from R12; Part Number (none) -> 1090
- U$2: Part Number (none) -> 1099
Connections:
- net +3.3V: now also U2.16 (VDD); no longer J10.3 (Pin_3), U$2.3V3
- net GND: now also U2.17 (GND); no longer J10.2 (Pin_2), U$2.GND
- net LOAD_CELL_DATA: no longer U$2.2
- net LOAD_CELL_SCK: no longer U$2.16/A2
- net MOTOR_ENABLE: no longer U$2.33/A14
- net STATUS_LED: no longer U$2.32/A13
- net BUTTON_LED: no longer names the net of U$2.14/A0
- net CHARGE_RELAY_CTRL: no longer names the net of U$2.29
- net HALL_EFFECT_SNS: no longer names the net of U$2.17/A3
- net HALL_EFFECT_SNS: no longer J10.1 (Pin_1)
- net LATCH_STAT: no longer names the net of U$2.31/A12
- net LED_RING: no longer names the net of U$2.39/A20
- net M1_DR1: no longer names the net of U$2.38/A19
- net M1_DR2: no longer names the net of U$2.37/A18
- net M1_EA: no longer names the net of U$2.3/CANTX
- net M1_EB: no longer names the net of U$2.4/CANRX
- net M2_DR1: no longer names the net of U$2.36/A17
- net M2_DR2: no longer names the net of U$2.35/A16
- net M2_EA: no longer names the net of U$2.5
- net M2_EB: no longer names the net of U$2.6
- net M3_DR1: no longer names the net of U$2.23/A9
- net M3_DR2: no longer names the net of U$2.22/A8
- net M3_EA: no longer names the net of U$2.24
- net M3_EB: no longer names the net of U$2.25
- net M4_DR1: no longer names the net of U$2.21/A7
- net M4_DR2: no longer names the net of U$2.20/A6
- net M4_EA: no longer names the net of U$2.26
- net M4_EB: no longer names the net of U$2.27
- net RX_JETSON: no longer names the net of U$2.7
- net SCL1: no longer names the net of U$2.19/A5/SCL
- net SDA1: no longer names the net of U$2.18/A4/SDA
- net TX_JETSON: no longer names the net of U$2.8
- net UNLATCH: no longer names the net of U$2.30
- net USB_SENSE: no longer names the net of U$2.34/A15

Commit message: rev 01 - fixing connectors
Parts:
- removed J11: Conn_01x03_Female, Connector_JST:JST_XH_B3B-XH-A_1x03_P2.50mm_Vertical, symbol Connector:Conn_01x03_Female
- removed J15: Conn_01x02_Female, TerminalBlock_4Ucon:TerminalBlock_4Ucon_1x02_P3.50mm_Horizontal, symbol Connector:Conn_01x02_Female
- added J11: Conn_01x04_Female, TerminalBlock_4Ucon:TerminalBlock_4Ucon_1x04_P3.50mm_Horizontal, symbol Connector:Conn_01x04_Female
Other:
- note added: "Charge INA219 I2C"
- note added: "Encoder 1"
- note added: "Encoder 2"
- note added: "Encoder 3"
- note added: "Encoder 4"
- note added: "LED Ring"
- note added: "LIDAR power"
- note added: "Load cell 1"
- note added: "Load cell 2"
- note added: "Main INA219 I2C"
- note added: "SEN-13879 Load Cell In"
- note added: "SEN-13879 SPI"
- note added: "Servo I2C"
- note added: "Servo power"
