File: pcb/bw_beer_caddy/bw_beer_caddy.kicad_sch (KiCad schematic)
At the start: 24 parts, among them J1 Conn_01x04_Female, J10 Conn_01x03_Female, J11 Conn_01x04_Female, J12 Conn_01x04_Female, J13 Conn_01x03_Female, J14 Conn_01x02_Female, J2 Conn_01x04_Female, J3 Conn_01x04_Female, J4 Conn_01x04_Female, J5 Conn_01x03_Female, J6 Conn_01x03_Female, J7 Conn_01x03_Female, J8 Conn_01x04_Female, J9 Conn_01x04_Female, U1 Pololu_5V_Step_Down_2851, U2 Pololu-MC33926-Dual-Motor, U3 Pololu-MC33926-Dual-Motor

Commit message: rev 01 pcb release
Parts:
- removed J10, J13: Conn_01x03_Female, Connector_JST:JST_XH_B3B-XH-A_1x03_P2.50mm_Vertical, symbol Connector:Conn_01x03_Female
- added J10, J13, J15: Conn_01x04_Female, Connector_JST:JST_PH_B4B-PH-K_1x04_P2.00mm_Vertical, symbol Connector:Conn_01x04_Female
- added J16: Conn_01x03_Female, Connector_JST:JST_PH_B3B-PH-K_1x03_P2.00mm_Vertical, symbol Connector:Conn_01x03_Female
- J1, J12, J2, J3, J4, J8, J9: footprint Connector_JST:JST_XH_B4B-XH-A_1x04_P2.50mm_Vertical -> Connector_JST:JST_PH_B4B-PH-K_1x04_P2.00mm_Vertical
- J5, J6, J7: footprint Connector_JST:JST_XH_B3B-XH-A_1x03_P2.50mm_Vertical -> Connector_JST:JST_PH_B3B-PH-K_1x03_P2.00mm_Vertical
Connections:
- net A+ is gone; now on net GRN: J6.3 (Pin_3)
- net A- is gone; now on net WHT: J5.3 (Pin_3)
- net E+ is gone; now on net RED: J5.1 (Pin_1), J6.2 (Pin_2)
- net E- is gone; now on net BLK: J5.2 (Pin_2), J6.1 (Pin_1)
- net MOTOR_ENABLE is gone; now on net MOTOR_EN: R2.2
- net +3.3V: now also J1.1 (Pin_1), J2.1 (Pin_1), J3.1 (Pin_1), J4.1 (Pin_1), J8.1 (Pin_1), J9.1 (Pin_1), U$2.3V3, U3.16 (VDD), J10.1 (Pin_1), J13.1 (Pin_1)
- net GND: now also J1.4 (Pin_4), J2.4 (Pin_4), J3.4 (Pin_4), J4.4 (Pin_4), J8.4 (Pin_4), J9.4 (Pin_4), U$2.GND, U$2.GND2, U2.12 (M1_PWM_D1), U2.3 (M2_PWM_D1), U2.7 (INV), U2.8 (SLEW), U3.12 (M1_PWM_D1), U3.17 (GND), U3.3 (M2_PWM_D1), U3.7 (INV), U3.8 (SLEW), J10.4 (Pin_4), J13.4 (Pin_4), J15.2 (Pin_2), J15.4 (Pin_4), J16.3 (Pin_3)
- net STATUS_LED: now also U$2.0/RX
- net MOTOR_EN: now reaches U$2.1/TX
- net MOTOR_EN: now also U2.9 (EN), U3.9 (EN)
- net M2_SPEED: now reaches U$2.10/CS
- net M2_SPEED: now also U2.4 (M2_PWM_D2)
- net M1_DIR+: now reaches U$2.11/MOSI
- net M1_DIR+: now also U2.14 (M1_IN1)
- net M1_DIR-: now reaches U$2.12/MISO
- net M1_DIR-: now also U2.15 (M1_IN2)
- net BUTTON_LED: now reaches U$2.14/A0
- net BUTTON_LED: now also J15.1 (Pin_1)
- net BUTTON_IN: now reaches U$2.15/A1
- net BUTTON_IN: now also J15.3 (Pin_3)
- net LOAD_CELL_CLK: now reaches U$2.16/A2
- net LOAD_CELL_CLK: now also J9.3 (Pin_3)
- net M2_SF: now reaches U$2.17/A3
- net M2_SF: now also U2.2 (M2_SF)
- net SDA1: now reaches U$2.18/A4/SDA
- net SDA1: now also J8.2 (Pin_2), J10.2 (Pin_2), J13.2 (Pin_2)
- net SCL1: now reaches U$2.19/A5/SCL
- net SCL1: now also J8.3 (Pin_3), J10.3 (Pin_3), J13.3 (Pin_3)
- net LOAD_CELL_DATA: now reaches U$2.2
- net LOAD_CELL_DATA: now also J9.2 (Pin_2)
- net M4_FB: now reaches U$2.20/A6
- net M4_FB: now also U3.1 (M2_FB)
- net M3_FB: now reaches U$2.21/A7
- net M3_FB: now also U3.10 (M1_FB)
- net M2_FB: now reaches U$2.22/A8
- net M2_FB: now also U2.1 (M2_FB)
- net M1_FB: now reaches U$2.23/A9
- net M1_FB: now also U2.10 (M1_FB)
- net EN3A: now reaches U$2.24
- net EN3A: now also J3.3 (Pin_3)
- net EN3B: now reaches U$2.25
- net EN3B: now also J3.2 (Pin_2)
- net EN4A: now reaches U$2.26
- net EN4A: now also J4.3 (Pin_3)
- net EN4B: now reaches U$2.27
- net EN4B: now also J4.2 (Pin_2)
- net M2_DIR+: now reaches U$2.28
- net M2_DIR+: now also U2.5 (M2_IN1)
- net M2_DIR-: now reaches U$2.29
- net M2_DIR-: now also U2.6 (M2_IN2)
- net EN1A: now reaches U$2.3/CANTX
- net EN1A: now also J1.3 (Pin_3)
- net M3_DIR+: now reaches U$2.30
- net M3_DIR+: now also U3.14 (M1_IN1)
- net M3_DIR-: now reaches U$2.31/A12
- net M3_DIR-: now also U3.15 (M1_IN2)
- net M1_SF: now reaches U$2.32/A13
- net M1_SF: now also U2.11 (M1_SF)
- net M4_SF: now reaches U$2.33/A14
- net M4_SF: now also U3.2 (M2_SF)
- net M4_DIR-: now reaches U$2.34/A15
- net M4_DIR-: now also U3.6 (M2_IN2)
- net M4_DIR+: now reaches U$2.35/A16
- net M4_DIR+: now also U3.5 (M2_IN1)
- net M4_SPEED: now reaches U$2.36/A17
- net M4_SPEED: now also U3.4 (M2_PWM_D2)
- net M3_SPEED: now reaches U$2.37/A18
- net M3_SPEED: now also U3.13 (M1_PWM_D2)
- net M3_SF: now reaches U$2.38/A19
- net M3_SF: now also U3.11 (M1_SF)
- net RING_DATA: now reaches U$2.39/A20
- net RING_DATA: now also J7.3 (Pin_3)
- net EN1B: now reaches U$2.4/CANRX
- net EN1B: now also J1.2 (Pin_2)
- net EN2A: now reaches U$2.5
- net EN2A: now also J2.3 (Pin_3)
- net EN2B: now reaches U$2.6
- net EN2B: now also J2.2 (Pin_2)
- net JETSON_RX: now reaches U$2.7
- net JETSON_RX: now also J16.2 (Pin_2)
- net JETSON_TX: now reaches U$2.8
- net JETSON_TX: now also J16.1 (Pin_1)
- net M1_SPEED: now reaches U$2.9/CS
- net M1_SPEED: now also U2.13 (M1_PWM_D2)
- net +5V: now reaches J11.1 (Pin_1)
- net +5V: now also J11.3 (Pin_3), J7.1 (Pin_1), U1.1 (OUT)
- net GND2: now reaches J11.2 (Pin_2)
- net GND2: now also J11.4 (Pin_4), J14.2 (Pin_2), J7.2 (Pin_2), U1.2 (GND)
- net RED: now reaches J12.1 (Pin_1)
- net BLK: now reaches J12.2 (Pin_2)
- net WHT: now reaches J12.3 (Pin_3)
- net GRN: now reaches J12.4 (Pin_4)
- net at U1.3 (VIN): now also J14.1 (Pin_1)
Other:
- note added: "A+"
- note added: "A-"
- note added: "BLUE"
- note added: "E+"
- note added: "E-"
- note added: "GREEN"
- note added: "YELLOW"
- moved on the sheet: J12, J2, J3, J4

Commit message: system test updates
Connections:
- net BLK renamed BLK/E-
- net GRN renamed GRN/A+
- net RED renamed RED/E+
- net WHT renamed WHT/A-
Changed lines of the file:
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@@
     (effects (font (size 1.27 1.27)) (justify left bottom))
   )
-  (label "GRN" (at 430.53 266.7 0)
+  (label "GRN{slash}A+" (at 430.53 266.7 0)
     (effects (font (size 1.27 1.27)) (justify left bottom))
   )
@@
     (effects (font (size 1.27 1.27)) (justify left bottom))
   )
-  (label "RED" (at 317.5 274.32 0)
+  (label "RED{slash}E+" (at 317.5 274.32 0)
     (effects (font (size 1.27 1.27)) (justify left bottom))
   )
@@
     (effects (font (size 1.27 1.27)) (justify left bottom))
   )
-  (label "GRN" (at 317.5 281.94 0)
+  (label "GRN{slash}A+" (at 317.5 281.94 0)
     (effects (font (size 1.27 1.27)) (justify left bottom))
   )
@@
     (effects (font (size 1.27 1.27)) (justify left bottom))
   )
-  (label "BLK" (at 430.53 261.62 0)
+  (label "BLK{slash}E-" (at 430.53 261.62 0)
     (effects (font (size 1.27 1.27)) (justify left bottom))
   )
@@
     (effects (font (size 1.27 1.27)) (justify left bottom))
   )
-  (label "RED" (at 430.53 259.08 0)
+  (label "RED{slash}E+" (at 430.53 259.08 0)
     (effects (font (size 1.27 1.27)) (justify left bottom))
   )
@@
     (effects (font (size 1.27 1.27)) (justify left bottom))
   )
-  (label "BLK" (at 317.5 276.86 0)
+  (label "BLK{slash}E-" (at 317.5 276.86 0)
     (effects (font (size 1.27 1.27)) (justify left bottom))
   )
@@
     (effects (font (size 1.27 1.27)) (justify left bottom))
   )
-  (label "WHT" (at 317.5 279.4 0)
+  (label "WHT{slash}A-" (at 317.5 279.4 0)
     (effects (font (size 1.27 1.27)) (justify left bottom))
   )
@@
     (effects (font (size 1.27 1.27)) (justify left bottom))
   )
-  (label "WHT" (at 430.53 264.16 0)
-    (effects (font (size 1.27 1.27)) (justify left bottom))
-  )
+  (label "WHT{slash}A-" (at 430.53 264.16 0)
+    (effects (font (size 1.27 1.27)) (justify left bottom))
+  )
