File: pcb/bw_beer_caddy/bw_beer_caddy.kicad_pcb (KiCad board)
At the start: 2 copper layers, 70 x 70 mm, 28 parts, among them J1 Conn_01x04_Female, J10 Conn_01x03_Female, J11 Conn_01x04_Female, J12 Conn_01x04_Female, J13 Conn_01x03_Female, J14 Conn_01x02_Female, J2 Conn_01x04_Female, J3 Conn_01x04_Female, J4 Conn_01x04_Female, J5 Conn_01x03_Female, J6 Conn_01x03_Female, J7 Conn_01x03_Female, J8 Conn_01x04_Female, J9 Conn_01x04_Female, U1 Pololu_5V_Step_Down_2851, U2 Pololu-MC33926-Dual-Motor, U3 Pololu-MC33926-Dual-Motor

Commit message: rev 01 pcb release
Parts:
- added J15: Conn_01x04_Female, Connector_JST:JST_PH_B4B-PH-K_1x04_P2.00mm_Vertical, F.Cu at (166.0, 63.8)
- added J16: Conn_01x03_Female, Connector_JST:JST_PH_B3B-PH-K_1x03_P2.00mm_Vertical, F.Cu at (132.7, 110.0)
- J1, J12, J2, J3, J4, J8, J9: footprint Connector_JST:JST_XH_B4B-XH-A_1x04_P2.50mm_Vertical -> Connector_JST:JST_PH_B4B-PH-K_1x04_P2.00mm_Vertical
- J10, J13: value Conn_01x03_Female -> Conn_01x04_Female; footprint Connector_JST:JST_XH_B3B-XH-A_1x03_P2.50mm_Vertical -> Connector_JST:JST_PH_B4B-PH-K_1x04_P2.00mm_Vertical
- J5, J6, J7: footprint Connector_JST:JST_XH_B3B-XH-A_1x03_P2.50mm_Vertical -> Connector_JST:JST_PH_B3B-PH-K_1x03_P2.00mm_Vertical
- moved J11 62.9 mm to (103.9, 56.4), turned to -90 degrees
- moved J7 46.7 mm to (115.8, 65.8), turned to 180 degrees
- moved J13 43.5 mm to (130.8, 102.5), turned to 0 degrees
- moved J10 43.3 mm to (166.0, 77.2), turned to 90 degrees
- moved J14 5.10 mm to (108.9, 74.0)
- moved J5 2.00 mm to (110.8, 110.0)
- moved J6 2.00 mm to (121.8, 110.0)
- moved D3 1.00 mm to (141.6, 45.6)
- moved R3 0.97 mm to (141.1, 49.0)
- moved J12 0.25 mm to (166.0, 90.8)
- moved J9 0.25 mm to (166.0, 104.2)
- renumbered REF** to HOLE1, REF** to HOLE2, REF** to HOLE3, REF** to HOLE4
Connections:
- J1 pad 1: unconnected-(J1-Pad1) -> +3.3V
- J1 pad 2: unconnected-(J1-Pad2) -> /EN1B
- J1 pad 3: unconnected-(J1-Pad3) -> /EN1A
- J1 pad 4: unconnected-(J1-Pad4) -> GND
- J10 pad 1: unconnected-(J10-Pad1) -> +3.3V
- J10 pad 2: unconnected-(J10-Pad2) -> /SDA1
- J10 pad 3: unconnected-(J10-Pad3) -> /SCL1
- J11 pad 1: unconnected-(J11-Pad1) -> +5V
- J11 pad 2: unconnected-(J11-Pad2) -> GND2
- J11 pad 3: unconnected-(J11-Pad3) -> +5V
- J11 pad 4: unconnected-(J11-Pad4) -> GND2
- J12 pad 1: unconnected-(J12-Pad1) -> /RED
- J12 pad 2: unconnected-(J12-Pad2) -> /BLK
- J12 pad 3: unconnected-(J12-Pad3) -> /WHT
- J12 pad 4: unconnected-(J12-Pad4) -> /GRN
- J13 pad 1: unconnected-(J13-Pad1) -> +3.3V
- J13 pad 2: unconnected-(J13-Pad2) -> /SDA1
- J13 pad 3: unconnected-(J13-Pad3) -> /SCL1
- J14 pad 1: unconnected-(J14-Pad1) -> Net-(J14-Pad1)
- J14 pad 2: unconnected-(J14-Pad2) -> GND2
- J2 pad 1: unconnected-(J2-Pad1) -> +3.3V
- J2 pad 2: unconnected-(J2-Pad2) -> /EN2B
- J2 pad 3: unconnected-(J2-Pad3) -> /EN2A
- J2 pad 4: unconnected-(J2-Pad4) -> GND
- J3 pad 1: unconnected-(J3-Pad1) -> +3.3V
- J3 pad 2: unconnected-(J3-Pad2) -> /EN3B
- J3 pad 3: unconnected-(J3-Pad3) -> /EN3A
- J3 pad 4: unconnected-(J3-Pad4) -> GND
- J4 pad 1: unconnected-(J4-Pad1) -> +3.3V
- J4 pad 2: unconnected-(J4-Pad2) -> /EN4B
- J4 pad 3: unconnected-(J4-Pad3) -> /EN4A
- J4 pad 4: unconnected-(J4-Pad4) -> GND
- J5 pad 1: /E+ -> /RED
- J5 pad 2: /E- -> /BLK
- J5 pad 3: /A- -> /WHT
- J6 pad 1: /E- -> /BLK
- J6 pad 2: /E+ -> /RED
- J6 pad 3: /A+ -> /GRN
- J7 pad 1: unconnected-(J7-Pad1) -> +5V
- J7 pad 2: unconnected-(J7-Pad2) -> GND2
- J7 pad 3: unconnected-(J7-Pad3) -> /RING_DATA
- J8 pad 1: unconnected-(J8-Pad1) -> +3.3V
- J8 pad 2: unconnected-(J8-Pad2) -> /SDA1
- J8 pad 3: unconnected-(J8-Pad3) -> /SCL1
- J8 pad 4: unconnected-(J8-Pad4) -> GND
- J9 pad 1: unconnected-(J9-Pad1) -> +3.3V
- J9 pad 2: unconnected-(J9-Pad2) -> /LOAD_CELL_DATA
- J9 pad 3: unconnected-(J9-Pad3) -> /LOAD_CELL_CLK
- J9 pad 4: unconnected-(J9-Pad4) -> GND
- R2 pad 2: /MOTOR_ENABLE -> /MOTOR_EN
- U$2 pad 0/RX: unconnected-(U$2-Pad0/RX) -> /STATUS_LED
- U$2 pad 1/TX: unconnected-(U$2-Pad1/TX) -> /MOTOR_EN
- U$2 pad 10/CS: unconnected-(U$2-Pad10/CS) -> /M2_SPEED
- U$2 pad 11/MOSI: unconnected-(U$2-Pad11/MOSI) -> /M1_DIR+
- U$2 pad 12/MISO: unconnected-(U$2-Pad12/MISO) -> /M1_DIR-
- U$2 pad 14/A0: unconnected-(U$2-Pad14/A0) -> /BUTTON_LED
- U$2 pad 15/A1: unconnected-(U$2-Pad15/A1) -> /BUTTON_IN
- U$2 pad 16/A2: unconnected-(U$2-Pad16/A2) -> /LOAD_CELL_CLK
- U$2 pad 17/A3: unconnected-(U$2-Pad17/A3) -> /M2_SF
- U$2 pad 18/A4/SDA: unconnected-(U$2-Pad18/A4/SDA) -> /SDA1
- U$2 pad 19/A5/SCL: unconnected-(U$2-Pad19/A5/SCL) -> /SCL1
- U$2 pad 2: unconnected-(U$2-Pad2) -> /LOAD_CELL_DATA
- U$2 pad 20/A6: unconnected-(U$2-Pad20/A6) -> /M4_FB
- U$2 pad 21/A7: unconnected-(U$2-Pad21/A7) -> /M3_FB
- U$2 pad 22/A8: unconnected-(U$2-Pad22/A8) -> /M2_FB
- U$2 pad 23/A9: unconnected-(U$2-Pad23/A9) -> /M1_FB
- U$2 pad 24: unconnected-(U$2-Pad24) -> /EN3A
- U$2 pad 25: unconnected-(U$2-Pad25) -> /EN3B
- U$2 pad 26: unconnected-(U$2-Pad26) -> /EN4A
- U$2 pad 27: unconnected-(U$2-Pad27) -> /EN4B
- U$2 pad 28: unconnected-(U$2-Pad28) -> /M2_DIR+
- U$2 pad 29: unconnected-(U$2-Pad29) -> /M2_DIR-
- U$2 pad 3/CANTX: unconnected-(U$2-Pad3/CANTX) -> /EN1A
- U$2 pad 30: unconnected-(U$2-Pad30) -> /M3_DIR+
- U$2 pad 31/A12: unconnected-(U$2-Pad31/A12) -> /M3_DIR-
- U$2 pad 32/A13: unconnected-(U$2-Pad32/A13) -> /M1_SF
- U$2 pad 33/A14: unconnected-(U$2-Pad33/A14) -> /M4_SF
- U$2 pad 34/A15: unconnected-(U$2-Pad34/A15) -> /M4_DIR-
- U$2 pad 35/A16: unconnected-(U$2-Pad35/A16) -> /M4_DIR+
- U$2 pad 36/A17: unconnected-(U$2-Pad36/A17) -> /M4_SPEED
- U$2 pad 37/A18: unconnected-(U$2-Pad37/A18) -> /M3_SPEED
- U$2 pad 38/A19: unconnected-(U$2-Pad38/A19) -> /M3_SF
- U$2 pad 39/A20: unconnected-(U$2-Pad39/A20) -> /RING_DATA
- U$2 pad 3V3: unconnected-(U$2-Pad3V3) -> +3.3V
- U$2 pad 4/CANRX: unconnected-(U$2-Pad4/CANRX) -> /EN1B
- U$2 pad 5: unconnected-(U$2-Pad5) -> /EN2A
- U$2 pad 6: unconnected-(U$2-Pad6) -> /EN2B
- U$2 pad 7: unconnected-(U$2-Pad7) -> /JETSON_RX
- U$2 pad 8: unconnected-(U$2-Pad8) -> /JETSON_TX
- U$2 pad 9/CS: unconnected-(U$2-Pad9/CS) -> /M1_SPEED
- U$2 pad GND: unconnected-(U$2-PadGND) -> GND
- U$2 pad GND2: unconnected-(U$2-PadGND2) -> GND
- U1 pad 1: unconnected-(U1-Pad1) -> +5V
- U1 pad 2: unconnected-(U1-Pad2) -> GND2
- U1 pad 3: unconnected-(U1-Pad3) -> Net-(J14-Pad1)
- U2 pad 1: unconnected-(U2-Pad1) -> /M2_FB
- U2 pad 10: unconnected-(U2-Pad10) -> /M1_FB
- U2 pad 11: unconnected-(U2-Pad11) -> /M1_SF
- U2 pad 12: unconnected-(U2-Pad12) -> GND
- U2 pad 13: unconnected-(U2-Pad13) -> /M1_SPEED
- U2 pad 14: unconnected-(U2-Pad14) -> /M1_DIR+
- U2 pad 15: unconnected-(U2-Pad15) -> /M1_DIR-
- U2 pad 2: unconnected-(U2-Pad2) -> /M2_SF
- U2 pad 3: unconnected-(U2-Pad3) -> GND
- U2 pad 4: unconnected-(U2-Pad4) -> /M2_SPEED
- U2 pad 5: unconnected-(U2-Pad5) -> /M2_DIR+
- U2 pad 6: unconnected-(U2-Pad6) -> /M2_DIR-
- U2 pad 7: unconnected-(U2-Pad7) -> GND
- U2 pad 8: unconnected-(U2-Pad8) -> GND
- U2 pad 9: unconnected-(U2-Pad9) -> /MOTOR_EN
- U3 pad 1: unconnected-(U3-Pad1) -> /M4_FB
- U3 pad 10: unconnected-(U3-Pad10) -> /M3_FB
- U3 pad 11: unconnected-(U3-Pad11) -> /M3_SF
- U3 pad 12: unconnected-(U3-Pad12) -> GND
- U3 pad 13: unconnected-(U3-Pad13) -> /M3_SPEED
- U3 pad 14: unconnected-(U3-Pad14) -> /M3_DIR+
- U3 pad 15: unconnected-(U3-Pad15) -> /M3_DIR-
- U3 pad 16: unconnected-(U3-Pad16) -> +3.3V
- U3 pad 17: unconnected-(U3-Pad17) -> GND
- U3 pad 2: unconnected-(U3-Pad2) -> /M4_SF
- U3 pad 3: unconnected-(U3-Pad3) -> GND
- U3 pad 4: unconnected-(U3-Pad4) -> /M4_SPEED
- U3 pad 5: unconnected-(U3-Pad5) -> /M4_DIR+
- U3 pad 6: unconnected-(U3-Pad6) -> /M4_DIR-
- U3 pad 7: unconnected-(U3-Pad7) -> GND
- U3 pad 8: unconnected-(U3-Pad8) -> GND
- U3 pad 9: unconnected-(U3-Pad9) -> /MOTOR_EN
Routing:
- net GND: track 0.00 -> 269.3 mm
- net +3.3V: track 0.00 -> 170.5 mm
- net /EN4B: track 0.00 -> 121.2 mm
- net /EN4A: track 0.00 -> 115.5 mm
- net /EN3B: track 0.00 -> 106.3 mm
- net /EN3A: track 0.00 -> 94.8 mm, vias 0 -> 1
- net /MOTOR_EN: track 0.00 -> 91.0 mm, vias 0 -> 1
- net /M3_DIR-: track 0.00 -> 80.2 mm
- net /SDA1: track 0.00 -> 77.9 mm
- net /WHT: track 0.00 -> 75.7 mm
- net /EN2B: track 0.00 -> 75.6 mm
- net /BLK: track 0.00 -> 75.5 mm
- net /EN1A: track 0.00 -> 75.2 mm
- net /SCL1: track 0.00 -> 74.4 mm
- net /RED: track 0.00 -> 74.1 mm
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- added copper zone on B.Cu, net (none)
- added copper zone on F.Cu, net (none)

Commit message: system test updates
Connections:
- net /BLK renamed /BLK/E-
- net /GRN renamed /GRN/A+
- net /RED renamed /RED/E+
- net /WHT renamed /WHT/A-
